Commit message: Add 1st version with gazebo simulation

File: src/motoman_hc10_support/urdf/hc10dtp_b00_macro.xacro (robot description, xacro)
@@ -3,6 +3,14 @@
   <xacro:macro name="motoman_hc10dtp_b00" params="prefix">
     <xacro:include filename="$(find motoman_resources)/urdf/common_materials.xacro"/>
+    <xacro:macro name="example_inertial" params="mass">
+      <inertial>
+        <origin xyz="0 0 0" rpy="0 0 0"/>
+        <mass value="${mass}"/>
+        <inertia ixx="0.1" ixy="0" ixz="0" iyy="0.1" iyz="0" izz="0.1"/>
+      </inertial>
+    </xacro:macro>
     <!-- link list -->
     <link name="${prefix}base_link">
+      <xacro:example_inertial mass="10.0"/>
       <visual>
         <geometry>
@@ -18,4 +26,5 @@
     </link>
     <link name="${prefix}link_1">
+      <xacro:example_inertial mass="10.0"/>
       <visual>
         <geometry>
@@ -31,4 +40,5 @@
     </link>
     <link name="${prefix}link_2">
+      <xacro:example_inertial mass="10.0"/>
       <visual>
         <geometry>
@@ -44,4 +54,5 @@
     </link>
     <link name="${prefix}link_3">
+      <xacro:example_inertial mass="10.0"/>
       <visual>
         <geometry>
@@ -57,4 +68,5 @@
     </link>
     <link name="${prefix}link_4">
+      <xacro:example_inertial mass="10.0"/>
       <visual>
         <geometry>
@@ -70,4 +82,5 @@
     </link>
     <link name="${prefix}link_5">
+      <xacro:example_inertial mass="10.0"/>
       <visual>
         <geometry>
@@ -83,4 +96,5 @@
     </link>
     <link name="${prefix}link_6">
+      <xacro:example_inertial mass="10.0"/>
       <visual>
         <geometry>
@@ -143,5 +157,7 @@
     <!-- end of joint list -->
     <!-- ROS-Industrial 'flange' frame: attachment point for EEF models -->
-    <link name="${prefix}flange"/>
+    <link name="${prefix}flange">
+      <xacro:example_inertial mass="0.01"/>
+    </link>
     <joint name="${prefix}joint_6-flange" type="fixed">
       <origin xyz="0.170 0 0" rpy="0 0 0"/>
@@ -150,5 +166,7 @@
     </joint>
     <!-- ROS-Industrial 'tool0' frame: all-zeros tool frame -->
-    <link name="${prefix}tool0"/>
+    <link name="${prefix}tool0">
+      <xacro:example_inertial mass="0.01"/>
+    </link>
     <joint name="${prefix}flange-tool0" type="fixed">
       <origin xyz="0 0 0" rpy="${radians(180)} ${radians(-90)} 0"/>
@@ -157,5 +175,7 @@
     </joint>
     <!-- ROS base_link to Robot Manufacturer World Coordinates transform -->
-    <link name="${prefix}base" />
+    <link name="${prefix}base">
+      <xacro:example_inertial mass="0.01"/>
+    </link>
     <joint name="${prefix}base_link-base" type="fixed">
       <origin xyz="0 0 0.275" rpy="0 0 0"/>

File: src/motoman_hc10dtp_b00_moveit2_config/config/motoman_hc10dtp_b00.urdf.xacro (robot description, xacro)
@@ -3,4 +3,4 @@
     <xacro:arg name="initial_positions_file" default="initial_positions.yaml" />
     <!-- Import motoman_hc10dtp_b00 urdf file -->
-    <xacro:include filename="$(find motoman_hc10_support)/urdf/hc10dtp_b00.urdf" />
+    <xacro:include filename="$(find motoman_hc10_support)/urdf/hc10dtp_b00.xacro" />
 </robot>
